File: hardware/Beacon_Lite/Beacon_Lite.kicad_sch (KiCad schematic)
At the start: 0 parts

Commit message: Started programming NUCLEO-H533 in VSCODE
* Able to use C++ and C
* Successful able to debug
* Can blink an LED when button is pressed via an interrupt.
Other:
- sheet FLED renamed FLED_Control
- sheet FLED_Control: file FLED.kicad_sch -> FLED_Control.kicad_sch
Changed lines of the file:
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@@
 			(color 0 0 0 0.0000)
 		)
-		(property "Sheetname" "FLED"
+		(property "Sheetname" "FLED_Control"
 			(at 65.405 17.0684 0)
 			(effects
@@
 			)
 		)
-		(property "Sheetfile" "FLED.kicad_sch"
+		(property "Sheetfile" "FLED_Control.kicad_sch"
 			(at 65.405 33.6046 0)
 			(effects
