File: hardware/Beacon_Tower/Beacon_Tower/FLED.kicad_sch (KiCad schematic)
At the start: 25 parts, among them U301 IS31FL3741

Commit message: Started assigning footprints. Tweaking schematic.
Parts:
- removed U301: IS31FL3741, symbol CUSTOM_SYMBOLS:IS31FL3741
- added U301: IS31FL3741, CUSTOM_FOOTPRINTS:QFN40P7X7_Thermal25, symbol CUSTOM_LIBRARY:IS31FL3741
- C301, C302, C303, C304, C305, C306: footprint Footprint_Library:0402_1005Metric_Handsolder -> Capacitor_SMD:C_0402_1005Metric
- R303, R304, R305, R306: footprint Footprint_Library:0402_1005Metric_Handsolder -> Resistor_SMD:R_0402_1005Metric
- TP301, TP302: footprint (none) -> TestPoint:TestPoint_Pad_D2.0mm
Connections:
- net CS1: now also U301.26 (CS1)
- net CS10: now also U301.35 (CS10)
- net CS11: now also U301.37 (CS11)
- net CS12: now also U301.38 (CS12)
- net CS13: now also U301.39 (CS13)
- net CS14: now also U301.40 (CS14)
- net CS15: now also U301.41 (CS15)
- net CS16: now also U301.42 (CS16)
- net CS17: now also U301.43 (CS17)
- net CS18: now also U301.44 (CS18)
- net CS19: now also U301.45 (CS19)
- net CS2: now also U301.27 (CS4)
- net CS20: now also U301.46 (CS20)
- net CS21: now also U301.47 (CS21)
- net CS22: now also U301.48 (CS22)
- net CS23: now also U301.49 (CS23)
- net CS24: now also U301.50 (CS24)
- net CS25: now also U301.51 (CS25)
- net CS26: now also U301.52 (CS26)
- net CS27: now also U301.53 (CS27)
- net CS28: now also U301.54 (CS28)
- net CS29: now also U301.56 (CS29)
- net CS3: now also U301.28 (CS3)
- net CS30: now also U301.57 (CS30)
- net CS31: now also U301.58 (CS31)
- net CS32: now also U301.59 (CS32)
- net CS33: now also U301.60 (CS33)
- net CS34: now also U301.1 (CS34)
- net CS35: now also U301.2 (CS35)
- net CS36: now also U301.3 (CS36)
- net CS37: now also U301.4 (CS37)
- net CS38: now also U301.5 (CS38)
- net CS39: now also U301.6 (CS39)
- net CS4: now also U301.27 (CS4)
- net CS5: now also U301.30 (CS5)
- net CS6: now also U301.31 (CS6)
- net CS7: now also U301.32 (CS7)
- net CS8: now also U301.33 (CS8)
- net CS9: now also U301.34 (CS9)
- net GND: now also R306.1, U301.12 (GND), U301.36 (GND), U301.55 (GND), U301.EP (GND)
- net I2C0_SCL: now also U301.10 (SCL)
- net I2C0_SDA: now also U301.9 (SDA)
- net SW1: now also U301.16 (SW1)
- net SW2: now also U301.17 (SW2)
- net SW3: now also U301.18 (SW3)
- net SW4: now also U301.19 (SW4)
- net SW5: now also U301.20 (SW5)
- net SW6: now also U301.21 (SW6)
- net SW7: now also U301.22 (SW7)
- net SW8: now also U301.23 (SW8)
- net VDD_1V8: no longer R306.2
- net VDD_4V5: now also U301.14 (AVCC), U301.15 (PVCC), U301.25 (PVCC)
- net at TP302.1: now also R306.2, U301.11 (SDB); no longer R306.1
- net at R304.2: now also U301.13 (ISET)
- net at R303.1, TP301.1: now also U301.7 (INTB)
- net at R305.2: now also U301.8 (ADDR)
Other:
- note added: "PU but have fet pull to gnd for reverse polarity"
- moved on the sheet: R306, TP302
