File: hardware/Beacon_Tower/Beacon_Tower/FLED_Array.kicad_sch (KiCad schematic)
At the start: 104 parts

Commit message: Started assigning footprints. Tweaking schematic.
Parts:
- removed D1388, D1396, D1404, D1412: ~, symbol CUSTOM_LIBRARY:RGB_CommAnode
- renumbered D1309 to D401, D1317 to D402, D1325 to D403, D1333 to D404, D1341 to D405, D1349 to D406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
Other:
- note added: "4 RGBs/Fret * (24 frets + open) = 100 RGBS (8 rows * 13 columns) - 4 RGBs = 100 RGBs"
- note added: "FLED Array"
